File: schematic/bd_mcu.sch (KiCad schematic (older format))
At the start: 2 parts

Commit message: wip
Parts:
- removed C1: C, symbol C
- removed U?: STM32F405, symbol STM32F405
- added U?: STM32F405ZG, symbol STM32F405ZG
Connections:
- net labels added: +3V3D
Changed lines of the file:
@@
-EESchema Schematic File Version 2  date Sat 19 Jan 2013 05:13:54 PM GMT
+EESchema Schematic File Version 2  date Thu 24 Jan 2013 06:08:02 PM GMT
+LIBS:aart_power_ports
 LIBS:aart_micros
 LIBS:aart_power_supplies
@@
 EELAYER 25  0
 EELAYER END
-$Descr A3 16535 11700
+$Descr A2 23400 16535
 encoding utf-8
 Sheet 1 1
 Title ""
-Date "19 jan 2013"
+Date "24 jan 2013"
 Rev ""
 Comp ""
@@
 $EndDescr
 $Comp
-L STM32F405 U?
-U 1 1 50FAD235
-P 5400 4450
-F 0 "U?" H 4550 5250 60  0000 L CNN
-F 1 "STM32F405" H 4550 5150 60  0000 L CNN
-	1    5400 4450
+L +3V3D #3V3D?
+U 1 1 5101787B
+P 4300 4600
+F 0 "#3V3D?" H 4325 4530 50  0000 L CNN
+F 1 "+3V3D" H 4165 4665 50  0000 L CNN
+	1    4300 4600
 	1    0    0    -1
 $EndComp
 $Comp
-L C C1
-U 1 1 50F858EF
-P 4450 4600
-F 0 "C1" H 4500 4700 50  0000 L CNN
-F 1 "C" H 4500 4500 50  0000 L CNN
-	1    4450 4600
+L STM32F405ZG U?
+U 1 1 510173FC
+P 7500 3300
+F 0 "U?" H 7800 3600 60  0000 L CNN
+F 1 "STM32F405ZG" H 7800 3500 60  0000 L CNN
+	1    7500 3300
 	1    0    0    -1
 $EndComp

Commit message: wip
Connections:
- net labels added: SRAM_A0, SRAM_A1, SRAM_A10, SRAM_A11, SRAM_A12, SRAM_A13, SRAM_A14, SRAM_A15, SRAM_A16, SRAM_A17, SRAM_A18, SRAM_A19, SRAM_A2, SRAM_A20, SRAM_A3, SRAM_A4, SRAM_A5, SRAM_A6, SRAM_A7, SRAM_A8, SRAM_A9, SRAM_D0, SRAM_D1, SRAM_D10, SRAM_D11, SRAM_D12, SRAM_D13, SRAM_D14, SRAM_D15, SRAM_D2, SRAM_D3, SRAM_D4, SRAM_D5, SRAM_D6, SRAM_D7, SRAM_D8, SRAM_D9, SRAM_~BHE~, SRAM_~BLE~, SRAM_~CS~, SRAM_~OE~, SRAM_~WE~
- wire segments 0 -> 42
Changed lines of the file:
@@
-EESchema Schematic File Version 2  date Thu 24 Jan 2013 06:08:02 PM GMT
+EESchema Schematic File Version 2  date Sun 27 Jan 2013 03:45:48 PM GMT
 LIBS:aart_power_ports
 LIBS:aart_micros
@@
 LIBS:contrib
 LIBS:valves
+LIBS:bd_mcu-cache
 EELAYER 25  0
 EELAYER END
@@
 Sheet 1 1
 Title ""
-Date "24 jan 2013"
+Date "25 jan 2013"
 Rev ""
 Comp ""
@@
 Comment4 ""
 $EndDescr
+Text HLabel 16200 4800 2    60   BiDi ~ 0
+SRAM_D12
+Text HLabel 16200 4700 2    60   BiDi ~ 0
+SRAM_D11
+Text HLabel 16200 4600 2    60   BiDi ~ 0
+SRAM_D10
+Text HLabel 16200 4500 2    60   BiDi ~ 0
+SRAM_D9
+Text HLabel 16200 4400 2    60   BiDi ~ 0
+SRAM_D8
+Text HLabel 16200 4300 2    60   BiDi ~ 0
+SRAM_D7
+Text HLabel 16200 4200 2    60   BiDi ~ 0
+SRAM_D6
+Text HLabel 16200 4100 2    60   BiDi ~ 0
+SRAM_D5
+Text HLabel 16200 4000 2    60   BiDi ~ 0
+SRAM_D4
+Wire Wire Line
+	15250 4800 16200 4800
+Wire Wire Line
+	15250 4600 16200 4600
+Wire Wire Line
+	15250 4400 16200 4400
+Wire Wire Line
+	15250 4200 16200 4200
+Wire Wire Line
+	7500 9400 6400 9400
+Wire Wire Line
+	7500 8500 6400 8500
+Wire Wire Line
+	6400 9900 7500 9900
+Wire Wire Line
+	15250 7700 16200 7700
+Wire Wire Line
+	7500 8900 6400 8900
+Wire Wire Line
+	15250 3300 16200 3300
+Wire Wire Line
+	15250 3600 16200 3600
+Wire Wire Line
+	7500 9600 6400 9600
+Wire Wire Line
+	15250 7200 16200 7200
+Wire Wire Line
+	15250 7000 16200 7000
+Wire Wire Line
+	15250 6800 16200 6800
+Wire Wire Line
+	15250 6500 16200 6500
+Wire Wire Line
+	15250 6300 16200 6300
+Wire Wire Line
+	15250 5500 16200 5500
+Wire Wire Line
+	15250 5300 16200 5300
+Wire Wire Line
+	15250 5100 16200 5100
+Wire Wire Line
+	15250 5000 16200 5000
+Wire Wire Line
+	15250 5200 16200 5200
+Wire Wire Line
+	15250 5400 16200 5400
+Wire Wire Line
+	15250 6200 16200 6200
+Wire Wire Line
+	15250 6400 16200 6400
+Wire Wire Line
+	15250 6700 16200 6700
+Wire Wire Line
+	15250 6900 16200 6900
+Wire Wire Line
+	15250 7100 16200 7100
+Wire Wire Line
+	7500 9500 6400 9500
+Wire Wire Line
+	7500 9700 6400 9700
+Wire Wire Line
+	15250 3700 16200 3700
+Wire Wire Line
+	15250 3400 16200 3400
+Wire Wire Line
+	7500 8800 6400 8800
+Wire Wire Line
+	7500 9800 6400 9800
+Wire Wire Line
+	7500 8400 6400 8400
+Wire Wire Line
+	7500 9200 6400 9200
+Wire Wire Line
+	7500 9300 6400 9300
+Wire Wire Line
+	15250 4000 16200 4000
+Wire Wire Line
+	15250 4100 16200 4100
+Wire Wire Line
+	15250 4300 16200 4300
+Wire Wire Line
+	15250 4500 16200 4500
+Wire Wire Line
+	15250 4700 16200 4700
+Text HLabel 6400 9400 0    60   BiDi ~ 0
+SRAM_D15
+Text HLabel 6400 9300 0    60   BiDi ~ 0
+SRAM_D14
+Text HLabel 6400 9200 0    60   BiDi ~ 0
+SRAM_D13
+Text HLabel 6400 8500 0    60   BiDi ~ 0
+SRAM_D3
+Text HLabel 6400 8400 0    60   BiDi ~ 0
+SRAM_D2
+Text HLabel 6400 9900 0    60   BiDi ~ 0
+SRAM_D1
+Text HLabel 6400 9800 0    60   BiDi ~ 0
+SRAM_D0
+Text HLabel 16200 7700 2    60   Output ~ 0
+SRAM_~CS~
+Text HLabel 6400 8900 0    60   Output ~ 0
+SRAM_~WE~
+Text HLabel 6400 8800 0    60   Output ~ 0
+SRAM_~OE~
+Text HLabel 16200 3400 2    60   Output ~ 0
+SRAM_~BHE~
+Text HLabel 16200 3300 2    60   Output ~ 0
+SRAM_~BLE~
+Text HLabel 16200 3700 2    60   Output ~ 0
+SRAM_A20
+Text HLabel 16200 3600 2    60   Output ~ 0
+SRAM_A19
+Text HLabel 6400 9700 0    60   Output ~ 0
+SRAM_A18
+Text HLabel 6400 9600 0    60   Output ~ 0
+SRAM_A17
+Text HLabel 6400 9500 0    60   Output ~ 0
+SRAM_A16
+Text HLabel 16200 7200 2    60   Output ~ 0
+SRAM_A15
+Text HLabel 16200 7100 2    60   Output ~ 0
+SRAM_A14
+Text HLabel 16200 7000 2    60   Output ~ 0
+SRAM_A13
+Text HLabel 16200 6900 2    60   Output ~ 0
+SRAM_A12
+Text HLabel 16200 6800 2    60   Output ~ 0
+SRAM_A11
+Text HLabel 16200 6700 2    60   Output ~ 0
+SRAM_A10
+Text HLabel 16200 6500 2    60   Output ~ 0
+SRAM_A9
+Text HLabel 16200 6400 2    60   Output ~ 0
+SRAM_A8
+Text HLabel 16200 6300 2    60   Output ~ 0
+SRAM_A7
+Text HLabel 16200 6200 2    60   Output ~ 0
+SRAM_A6
+Text HLabel 16200 5500 2    60   Output ~ 0
+SRAM_A5
+Text HLabel 16200 5400 2    60   Output ~ 0
+SRAM_A4
+Text HLabel 16200 5300 2    60   Output ~ 0
+SRAM_A3
+Text HLabel 16200 5200 2    60   Output ~ 0
+SRAM_A2
+Text HLabel 16200 5100 2    60   Output ~ 0
+SRAM_A1
+Text HLabel 16200 5000 2    60   Output ~ 0
+SRAM_A0
 $Comp
 L +3V3D #3V3D?
 U 1 1 5101787B
 P 4300 4600
-F 0 "#3V3D?" H 4325 4530 50  0000 L CNN
+F 0 "#3V3D?" H 4325 4530 50  0001 L CNN
 F 1 "+3V3D" H 4165 4665 50  0000 L CNN
 	1    4300 4600

Commit message: wip
Parts:
- added X?: 8MHz, symbol CRYSTAL
Connections:
- net labels added: 0VD
- wire segments 42 -> 52
Changed lines of the file:
@@
-EESchema Schematic File Version 2  date Sun 27 Jan 2013 03:45:48 PM GMT
+EESchema Schematic File Version 2  date 28/01/2013 12:58:48
 LIBS:aart_power_ports
 LIBS:aart_micros
@@
 Sheet 1 1
 Title ""
-Date "25 jan 2013"
+Date "28 jan 2013"
 Rev ""
 Comp ""
@@
 Comment4 ""
 $EndDescr
+Connection ~ 15450 11900
+Wire Wire Line
+	15250 11900 15450 11900
+Connection ~ 15450 11700
+Wire Wire Line
+	15250 11700 15450 11700
+Connection ~ 15450 11500
+Wire Wire Line
+	15250 11500 15450 11500
+Connection ~ 15450 11300
+Wire Wire Line
+	15250 11300 15450 11300
+Wire Wire Line
+	15250 11100 15450 11100
+Wire Wire Line
+	15450 11100 15450 11950
+Wire Wire Line
+	15250 4700 16200 4700
+Wire Wire Line
+	15250 4500 16200 4500
+Wire Wire Line
+	15250 4300 16200 4300
+Wire Wire Line
+	15250 4100 16200 4100
+Wire Wire Line
+	15250 4000 16200 4000
+Wire Wire Line
+	7500 9300 6400 9300
+Wire Wire Line
+	7500 9200 6400 9200
+Wire Wire Line
+	7500 8400 6400 8400
+Wire Wire Line
+	7500 9800 6400 9800
+Wire Wire Line
+	7500 8800 6400 8800
+Wire Wire Line
+	15250 3400 16200 3400
+Wire Wire Line
+	15250 3700 16200 3700
+Wire Wire Line
+	7500 9700 6400 9700
+Wire Wire Line
+	7500 9500 6400 9500
+Wire Wire Line
+	15250 7100 16200 7100
+Wire Wire Line
+	15250 6900 16200 6900
+Wire Wire Line
+	15250 6700 16200 6700
+Wire Wire Line
+	15250 6400 16200 6400
+Wire Wire Line
+	15250 6200 16200 6200
+Wire Wire Line
+	15250 5400 16200 5400
+Wire Wire Line
+	15250 5200 16200 5200
+Wire Wire Line
+	15250 5000 16200 5000
+Wire Wire Line
+	15250 5100 16200 5100
+Wire Wire Line
+	15250 5300 16200 5300
+Wire Wire Line
+	15250 5500 16200 5500
+Wire Wire Line
+	15250 6300 16200 6300
+Wire Wire Line
+	15250 6500 16200 6500
+Wire Wire Line
+	15250 6800 16200 6800
+Wire Wire Line
+	15250 7000 16200 7000
+Wire Wire Line
+	15250 7200 16200 7200
+Wire Wire Line
+	7500 9600 6400 9600
+Wire Wire Line
+	15250 3600 16200 3600
+Wire Wire Line
+	15250 3300 16200 3300
+Wire Wire Line
+	7500 8900 6400 8900
+Wire Wire Line
+	15250 7700 16200 7700
+Wire Wire Line
+	6400 9900 7500 9900
+Wire Wire Line
+	7500 8500 6400 8500
+Wire Wire Line
+	7500 9400 6400 9400
+Wire Wire Line
+	15250 4200 16200 4200
+Wire Wire Line
+	15250 4400 16200 4400
+Wire Wire Line
+	15250 4600 16200 4600
+Wire Wire Line
+	15250 4800 16200 4800
+Wire Wire Line
+	15250 11200 15450 11200
+Connection ~ 15450 11200
+Wire Wire Line
+	15250 11400 15450 11400
+Connection ~ 15450 11400
+Wire Wire Line
+	15250 11600 15450 11600
+Connection ~ 15450 11600
+Wire Wire Line
+	15250 11800 15450 11800
+Connection ~ 15450 11800
+$Comp
+L 0VD #0VD?
+U 1 1 510674AC
+P 15450 12100
+F 0 "#0VD?" H 15510 12215 50  0001 L CNN
+F 1 "0VD" H 15380 12040 50  0000 L CNN
+	1    15450 12100
+	1    0    0    -1
+$EndComp
+$Comp
+L +3V3D #3V3D?
+U 1 1 5106749A
+P 6700 11000
+F 0 "#3V3D?" H 6725 10930 50  0000 L CNN
+F 1 "+3V3D" H 6565 11065 50  0000 L CNN
+	1    6700 11000
+	1    0    0    -1
+$EndComp
+$Comp
+L CRYSTAL X?
+U 1 1 510670E9
+P 17050 8650
+F 0 "X?" V 17100 8400 60  0000 C CNN
+F 1 "8MHz" V 16850 8350 60  0000 C CNN
+	1    17050 8650
+	0    -1   -1   0
+$EndComp
 Text HLabel 16200 4800 2    60   BiDi ~ 0
 SRAM_D12
@@
 Text HLabel 16200 4000 2    60   BiDi ~ 0
 SRAM_D4
-Wire Wire Line
-	15250 4800 16200 4800
-Wire Wire Line
-	15250 4600 16200 4600
-Wire Wire Line
-	15250 4400 16200 4400
-Wire Wire Line
-	15250 4200 16200 4200
-Wire Wire Line
-	7500 9400 6400 9400
-Wire Wire Line
-	7500 8500 6400 8500
-Wire Wire Line
-	6400 9900 7500 9900
-Wire Wire Line
-	15250 7700 16200 7700
-Wire Wire Line
-	7500 8900 6400 8900
-Wire Wire Line
-	15250 3300 16200 3300
-Wire Wire Line
-	15250 3600 16200 3600
-Wire Wire Line
-	7500 9600 6400 9600
-Wire Wire Line
-	15250 7200 16200 7200
-Wire Wire Line
-	15250 7000 16200 7000
-Wire Wire Line
-	15250 6800 16200 6800
-Wire Wire Line
-	15250 6500 16200 6500
-Wire Wire Line
-	15250 6300 16200 6300
-Wire Wire Line
-	15250 5500 16200 5500
-Wire Wire Line
-	15250 5300 16200 5300
-Wire Wire Line
-	15250 5100 16200 5100
-Wire Wire Line
-	15250 5000 16200 5000
-Wire Wire Line
-	15250 5200 16200 5200
-Wire Wire Line
-	15250 5400 16200 5400
-Wire Wire Line
-	15250 6200 16200 6200
-Wire Wire Line
-	15250 6400 16200 6400
-Wire Wire Line
-	15250 6700 16200 6700
-Wire Wire Line
-	15250 6900 16200 6900
-Wire Wire Line
-	15250 7100 16200 7100
-Wire Wire Line
-	7500 9500 6400 9500
-Wire Wire Line
-	7500 9700 6400 9700
-Wire Wire Line
-	15250 3700 16200 3700
-Wire Wire Line
-	15250 3400 16200 3400
-Wire Wire Line
-	7500 8800 6400 8800
-Wire Wire Line
-	7500 9800 6400 9800
-Wire Wire Line
-	7500 8400 6400 8400
-Wire Wire Line
-	7500 9200 6400 9200
-Wire Wire Line
-	7500 9300 6400 9300
-Wire Wire Line
-	15250 4000 16200 4000
-Wire Wire Line
-	15250 4100 16200 4100
-Wire Wire Line
-	15250 4300 16200 4300
-Wire Wire Line
-	15250 4500 16200 4500
-Wire Wire Line
-	15250 4700 16200 4700
 Text HLabel 6400 9400 0    60   BiDi ~ 0
 SRAM_D15
@@
 SRAM_A0
 $Comp
-L +3V3D #3V3D?
-U 1 1 5101787B
-P 4300 4600
-F 0 "#3V3D?" H 4325 4530 50  0001 L CNN
-F 1 "+3V3D" H 4165 4665 50  0000 L CNN
-	1    4300 4600
-	1    0    0    -1
-$EndComp
-$Comp
 L STM32F405ZG U?

Commit message: wip
Parts:
- added C? (x12): 100n, symbol C
- gave numbers to parts that had none: 2
Connections:
- wire segments 52 -> 94

Commit message: wip
Parts:
- added C? (x2): 20p, symbol C
- added C? (x2): 6p8, symbol C
- added C? (x3): 100n, symbol C
- added C? (x2): 2u2, symbol C
- added C? (x3): 1u, symbol C
- added L?: ferrite 0603, symbol INDUCTOR
- added R?: 220, symbol R
- added R? (x3): 0, symbol R
- added R?: 47, symbol R
- added X?: 32.768kHz, symbol CRYSTAL
Connections:
- net labels added: +VBAT
- wire segments 94 -> 146
