File: schematic/bd_mcu.sch (KiCad schematic (older format))
At the start: 33 parts, among them U1 STM32F405ZG, X1 8MHz

Commit message: wip
Connections:
- wire segments 146 -> 148

Commit message: wip
Parts:
- added U?: R1LV1616R, symbol R1LV1616R
Changed lines of the file:
@@
-EESchema Schematic File Version 2  date 14/02/2013 07:51:00
+EESchema Schematic File Version 2  date 22/02/2013 13:27:21
 LIBS:aart_connectors
 LIBS:aart_micros
@@
 Sheet 1 1
 Title ""
-Date "14 feb 2013"
+Date "22 feb 2013"
 Rev ""
 Comp ""
@@
 Comment4 ""
 $EndDescr
+$Comp
+L R1LV1616R U?
+U 1 1 51273732
+P 17500 6600
+F 0 "U?" H 17800 6900 60  0000 L CNN
+F 1 "R1LV1616R" H 17800 6800 60  0000 L CNN
+F 3 "http://documentation.renesas.com/doc/products/memory/rej03c0101_r1lv1616r.pdf" H 18700 7050 60  0001 C CNN
+	1    17500 6600
+	1    0    0    -1
+$EndComp
 Wire Wire Line
 	2900 10300 2900 10100

Commit message: added SRAM to MCU and analogue in sheet
Parts:
- added C? (x2): 100n, symbol C
- added LED?: GREEN, symbol LED
- added LED?: RED, symbol LED
- added PL?: ARM_10_PIN_MICRO_HEADER, symbol ARM_10_PIN_MICRO_HEADER
- added R? (x2): 1k, symbol R
- added U?: R1LV1616R, symbol R1LV1616R
Connections:
- net labels added: A0, A1, A10, A11, A12, A13, A14, A15, A16, A17, A18, A19, A2, A3, A4, A5, A6, A7, A8, A9, D0, D1, D10, D11, D12, D13, D14, D15, D2, D3, D4, D5, D6, D7, D8, D9, JTAG-SWCLK, JTAG-SWDIO, SRAM_~CS1~, SRAM_~CS2~, ~BHE~, ~BLE~, ~OE~, ~WE~
- net labels removed: SRAM_A0, SRAM_A1, SRAM_A10, SRAM_A11, SRAM_A12, SRAM_A13, SRAM_A14, SRAM_A15, SRAM_A16, SRAM_A17, SRAM_A18, SRAM_A19, SRAM_A2, SRAM_A20, SRAM_A3, SRAM_A4, SRAM_A5, SRAM_A6, SRAM_A7, SRAM_A8, SRAM_A9, SRAM_D0, SRAM_D1, SRAM_D10, SRAM_D11, SRAM_D12, SRAM_D13, SRAM_D14, SRAM_D15, SRAM_D2, SRAM_D3, SRAM_D4, SRAM_D5, SRAM_D6, SRAM_D7, SRAM_D8, SRAM_D9, SRAM_~BHE~, SRAM_~BLE~, SRAM_~CS~, SRAM_~OE~, SRAM_~WE~
- wire segments 148 -> 263

Commit message: started analogue in
Connections:
- net labels added: LO
- wire segments 263 -> 264
