File: schematic/bd_psu.sch (KiCad schematic (older format))
At the start: 2 parts

Commit message: wip
Parts:
- added C?: CPOL, symbol CPOL
Changed lines of the file:
@@
-EESchema Schematic File Version 2  date Tuesday, 15 January 2013 22:02:56
+EESchema Schematic File Version 2  date 16/01/2013 15:22:48
+LIBS:aart_power_supplies
+LIBS:aart_connectors
+LIBS:aart_passives
 LIBS:power
 LIBS:device
@@
 LIBS:cypress
 LIBS:siliconi
-LIBS:connectors
 LIBS:opto
 LIBS:atmel
 LIBS:contrib
 LIBS:valves
-LIBS:power_supplies
-LIBS:passives
-LIBS:bd_psu-cache
-EELAYER 27 0
+EELAYER 25  0
 EELAYER END
-$Descr A3 16535 11693
+$Descr A3 16535 11700
 encoding utf-8
 Sheet 1 1
 Title ""
-Date "15 jan 2013"
+Date "16 jan 2013"
 Rev ""
 Comp ""
@@
 $EndDescr
 $Comp
+L CPOL C?
+U 1 1 50F6C598
+P 8450 6200
+F 0 "C?" H 8600 6350 50  0000 L CNN
+F 1 "CPOL" H 8600 6250 50  0000 L CNN
+	1    8450 6200
+	1    0    0    -1
+$EndComp
+$Comp
 L LTC4160 U?

Commit message: wip
Parts:
- removed C?: CPOL, symbol CPOL
- added C1: C, symbol C
- gave numbers to parts that had none: 2
Connections:
- wire segments 0 -> 5
Changed lines of the file:
@@
-EESchema Schematic File Version 2  date 16/01/2013 15:22:48
+EESchema Schematic File Version 2  date Thursday, 17 January 2013 20:16:58
 LIBS:aart_power_supplies
 LIBS:aart_connectors
@@
 LIBS:contrib
 LIBS:valves
-EELAYER 25  0
+LIBS:bd_psu-cache
+EELAYER 27 0
 EELAYER END
-$Descr A3 16535 11700
+$Descr A3 16535 11693
 encoding utf-8
 Sheet 1 1
 Title ""
-Date "16 jan 2013"
+Date "17 jan 2013"
 Rev ""
 Comp ""
@@
 $EndDescr
 $Comp
-L CPOL C?
-U 1 1 50F6C598
-P 8450 6200
-F 0 "C?" H 8600 6350 50  0000 L CNN
-F 1 "CPOL" H 8600 6250 50  0000 L CNN
-	1    8450 6200
-	1    0    0    -1
-$EndComp
-$Comp
-L LTC4160 U?
+L LTC4160 U1
 U 1 1 50F5B486
 P 6400 4150
-F 0 "U?" H 6700 4450 60  0000 L CNN
+F 0 "U1" H 6700 4450 60  0000 L CNN
 F 1 "LTC4160" H 6700 4350 60  0000 L CNN
 	1    6400 4150
@@
 $EndComp
 $Comp
-L R R?
+L R R1
 U 1 1 50F5BB5F
-P 7200 6600
-F 0 "R?" H 7280 6700 50  0000 L TNN
-F 1 "R" H 7300 6600 50  0000 L TNN
-	1    7200 6600
+P 7200 6300
+F 0 "R1" H 7280 6400 50  0000 L TNN
+F 1 "R" H 7300 6300 50  0000 L TNN
+	1    7200 6300
 	1    0    0    -1
 $EndComp
+Wire Wire Line
+	7200 6050 7200 5950
+Wire Wire Line
+	7200 6550 7600 6550
+Wire Wire Line
+	7600 6550 7600 5950
+$Comp
+L C C1
+U 1 1 50F858EF
+P 5850 4550
+F 0 "C1" H 5900 4650 50  0000 L CNN
+F 1 "C" H 5900 4450 50  0000 L CNN
+	1    5850 4550
+	1    0    0    -1
+$EndComp
+Wire Wire Line
+	5850 4350 5850 4150
+Wire Wire Line
+	5850 4150 6400 4150
 $EndSCHEMATC

Commit message: wip
Parts:
- removed U1: LTC4160, symbol LTC4160
- added U?: LTC3538, symbol LTC3538
Changed lines of the file:
@@
-EESchema Schematic File Version 2  date Thursday, 17 January 2013 20:16:58
+EESchema Schematic File Version 2  date 12/02/2013 16:45:36
 LIBS:aart_power_supplies
 LIBS:aart_connectors
@@
 LIBS:valves
 LIBS:bd_psu-cache
-EELAYER 27 0
+EELAYER 25  0
 EELAYER END
-$Descr A3 16535 11693
+$Descr A3 16535 11700
 encoding utf-8
 Sheet 1 1
 Title ""
-Date "17 jan 2013"
+Date "12 feb 2013"
 Rev ""
 Comp ""
@@
 $EndDescr
 $Comp
-L LTC4160 U1
-U 1 1 50F5B486
-P 6400 4150
-F 0 "U1" H 6700 4450 60  0000 L CNN
-F 1 "LTC4160" H 6700 4350 60  0000 L CNN
-	1    6400 4150
+L LTC3538 U?
+U 1 1 511A3F6B
+P 8800 4500
+F 0 "U?" H 8800 4650 60  0000 L CNN
+F 1 "LTC3538" H 8800 4550 60  0000 L CNN
+	1    8800 4500
 	1    0    0    -1
 $EndComp

Commit message: wip
Parts:
- added C?: 330pF, symbol C
- added C?: 33pF, symbol C
- added C?: 22uF, symbol C
- added C?: 10u, symbol C
- added C?: 100n, symbol C
- added L?: 3.3uH, symbol INDUCTOR
- added L?: ?, symbol INDUCTOR
- added R?: 10k, symbol R
- added R?: 200k, symbol R
- added R?: 15k, symbol R
- added ST?: STAR-2, symbol STAR-2
- C1: value C -> 10uF
- R1: value R -> 464k
Connections:
- net labels added: +3V3A, +3V3D, +V_BAT_OR_USB, 0VA, 0VD
- wire segments 5 -> 36
Other:
- note added: "2.9V to 5.5V"
- note added: "is this cap needed?"
