File: schematic/bd_usb_otg.sch (KiCad schematic (older format))
At the start: 2 parts

Commit message: wip
Connections:
- net labels added: 0VD
- wire segments 0 -> 14
Changed lines of the file:
@@
-EESchema Schematic File Version 2  date 30/01/2013 13:12:58
+EESchema Schematic File Version 2  date 04/02/2013 16:38:08
 LIBS:aart_connectors
 LIBS:aart_micros
@@
 LIBS:contrib
 LIBS:valves
+LIBS:bd_usb_otg-cache
 EELAYER 25  0
 EELAYER END
@@
 Sheet 1 1
 Title ""
-Date "30 jan 2013"
+Date "4 feb 2013"
 Rev ""
 Comp ""
@@
 $EndDescr
 $Comp
+L 0VD #PWR?
+U 1 1 510FD489
+P 13700 3750
+F 0 "#PWR?" H 13760 3865 50  0001 L CNN
+F 1 "0VD" H 13630 3690 50  0000 L CNN
+	1    13700 3750
+	1    0    0    -1
+$EndComp
+Wire Wire Line
+	13700 3600 13700 3500
+Connection ~ 14150 4450
+Wire Wire Line
+	14150 3500 14150 4450
+Connection ~ 13850 4250
+Wire Wire Line
+	13850 3500 13850 4250
+Wire Wire Line
+	14700 4950 14700 4550
+Wire Wire Line
+	14700 4550 14900 4550
+Wire Wire Line
+	13300 4350 14900 4350
+Wire Wire Line
+	14900 4150 14500 4150
+Wire Wire Line
+	14900 4250 13450 4250
+Wire Wire Line
+	14900 4450 13150 4450
+Wire Wire Line
+	14900 4700 14700 4700
+Connection ~ 14700 4700
+Wire Wire Line
+	14000 3500 14000 4350
+Connection ~ 14000 4350
+Wire Wire Line
+	14500 4150 14500 2600
+Wire Wire Line
+	14500 2600 13850 2600
+Wire Wire Line
+	13850 2600 13850 2750
+$Comp
+L 0VD #PWR?
+U 1 1 510FD248
+P 14700 4950
+F 0 "#PWR?" H 14760 5065 50  0001 L CNN
+F 1 "0VD" H 14630 4890 50  0000 L CNN
+	1    14700 4950
+	1    0    0    -1
+$EndComp
+$Comp
 L USB_MICRO_AB PL?
 U 1 1 510830E0
-P 14400 4100
-F 0 "PL?" H 14580 4370 50  0000 L BNN
-F 1 "USB_MICRO_AB" H 14910 4290 60  0000 C CNN
-	1    14400 4100
+P 14900 4150
+F 0 "PL?" H 15080 4420 50  0000 L BNN
+F 1 "USB_MICRO_AB" H 15410 4340 60  0000 C CNN
+	1    14900 4150
 	1    0    0    -1
 $EndComp
@@
 L VBUS053AZ-HAF IC?
 U 1 1 5108343E
-P 11300 4850
-F 0 "IC?" H 11450 5200 60  0000 C CNN
-F 1 "VBUS053AZ-HAF" H 11750 5300 60  0000 C CNN
-	1    11300 4850
-	1    0    0    -1
+P 13850 3500
+F 0 "IC?" H 14000 3850 60  0000 C CNN
+F 1 "VBUS053AZ-HAF" H 14300 3950 60  0000 C CNN
+	1    13850 3500
+	0    -1   -1   0
 $EndComp
 $EndSCHEMATC

Commit message: wip
Parts:
- added C?: 10u, symbol C
- added C?: 22u, symbol C
- added C?: C, symbol C
- added L?: 3u3H, symbol INDUCTOR
- added Q?: SI2333DS, symbol SI2333DS
- added R? (x3): R, symbol R
- added U?: LTC4160, symbol LTC4160
Connections:
- net labels added: +5V_USB, +VBAT, 0VBAT, BAT_THERM, USB_D+, USB_D-
- wire segments 14 -> 48

Commit message: wip
Parts:
- removed Q?: SI2333DS, symbol SI2333DS
- C?: value C -> 100n
- R?: value R -> 3k01
- R?: value R -> 1k
- R?: value R -> 100k
Connections:
- net labels added: BAT_CHARGE, BAT_PWR_FAULT, ENABLE_USB_OTH, USB_ID, USB_VBUS_GOOD
- wire segments 48 -> 52
Changed lines of the file:
@@
-EESchema Schematic File Version 2  date 07/02/2013 16:43:40
+EESchema Schematic File Version 2  date 11/02/2013 16:05:40
 LIBS:aart_connectors
 LIBS:aart_micros
@@
 Sheet 1 1
 Title ""
-Date "7 feb 2013"
+Date "11 feb 2013"
 Rev ""
 Comp ""
@@
 Comment4 ""
 $EndDescr
+Wire Wire Line
+	5750 3900 9000 3900
+Wire Wire Line
+	6800 6100 6800 5900
+Wire Wire Line
+	6800 8300 9850 8300
+Wire Wire Line
+	9000 5900 10000 5900
+Wire Wire Line
+	9000 6300 10300 6300
+Wire Wire Line
+	10000 5900 10000 5850
+Connection ~ 7500 8300
+Wire Wire Line
+	7500 8100 7500 8300
+Wire Wire Line
+	9800 5400 9800 5500
+Wire Wire Line
+	5750 3800 9000 3800
+Connection ~ 7900 7350
+Wire Wire Line
+	7100 7350 9250 7350
+Wire Wire Line
+	9850 8300 9850 7100
+Wire Wire Line
+	8550 7650 8550 7550
+Wire Wire Line
+	8550 7550 8300 7550
+Wire Wire Line
+	8300 7550 8300 7200
+Wire Wire Line
+	10300 6600 9000 6600
+Wire Wire Line
+	8100 7650 8100 7200
+Connection ~ 9800 5400
+Wire Wire Line
+	9700 5400 10000 5400
+Wire Wire Line
+	10000 5400 10000 5450
+Wire Wire Line
+	9000 5400 9100 5400
+Connection ~ 6800 5400
+Wire Wire Line
+	6800 5500 6800 5300
+Connection ~ 8600 2050
+Wire Wire Line
+	8600 2000 8600 3600
+Wire Wire Line
+	7950 2200 7950 2050
+Wire Wire Line
+	7950 2050 8600 2050
+Connection ~ 8100 3800
+Wire Wire Line
+	8100 2950 8100 3800
+Connection ~ 8800 4150
+Wire Wire Line
+	9000 4150 8800 4150
+Wire Wire Line
+	8600 3600 9000 3600
+Wire Wire Line
+	9000 4000 8800 4000
+Wire Wire Line
+	8800 4000 8800 4400
+Wire Wire Line
+	7950 2950 7950 3700
+Connection ~ 7950 3700
+Wire Wire Line
+	8250 2950 8250 3900
+Connection ~ 8250 3900
+Wire Wire Line
+	7800 3050 7800 2950
+Wire Wire Line
+	6800 5400 7100 5400
+Wire Wire Line
+	9800 5500 9000 5500
+Wire Wire Line
+	7100 6600 6800 6600
+Wire Wire Line
+	8550 8300 8550 8150
+Wire Wire Line
+	8100 8150 8100 8300
+Connection ~ 8100 8300
+Wire Wire Line
+	9850 7100 10300 7100
+Connection ~ 8550 8300
+Wire Wire Line
+	7500 7700 7500 7550
+Connection ~ 8100 7550
+Wire Wire Line
+	7900 7350 7900 7200
+Wire Wire Line
+	9250 7350 9250 6850
+Wire Wire Line
+	9250 6850 10300 6850
+Wire Wire Line
+	7100 6850 7100 6800
+Wire Wire Line
+	5750 3700 9000 3700
+Wire Wire Line
+	9000 5700 9250 5700
+Wire Wire Line
+	9250 5700 9250 5500
 Connection ~ 9250 5500
 Wire Wire Line
-	9250 5500 9250 5700
-Wire Wire Line
-	9250 5700 9000 5700
-Wire Wire Line
-	5750 3700 9000 3700
-Wire Wire Line
-	7100 6850 7100 6800
-Wire Wire Line
-	10300 6850 9250 6850
-Wire Wire Line
-	9250 6850 9250 7350
-Wire Wire Line
-	7900 7350 7900 7200
-Connection ~ 8100 7550
-Wire Wire Line
-	8100 7550 7800 7550
-Wire Wire Line
-	7800 7550 7800 7700
-Connection ~ 8550 8300
-Wire Wire Line
-	10300 7100 9850 7100
-Wire Wire Line
-	6450 8300 9850 8300
-Connection ~ 6450 8300
-Wire Wire Line
-	6450 8400 6450 6000
-Connection ~ 8100 8300
-Wire Wire Line
-	8100 8150 8100 8300
-Wire Wire Line
-	8550 8300 8550 8150
-Wire Wire Line
-	7100 6600 6800 6600
-Wire Wire Line
-	10000 6000 9000 6000
-Wire Wire Line
-	9000 5500 9800 5500
+	7500 7550 8100 7550
+Wire Wire Line
+	10300 6400 9000 6400
+Wire Wire Line
+	10300 6200 9000 6200
+Wire Wire Line
+	9450 5950 9450 5900
+Connection ~ 9450 5900
+Wire Wire Line
+	6800 6600 6800 8400
+Connection ~ 6800 8300
+Wire Wire Line
+	7100 6000 6800 6000
 Connection ~ 6800 6000
 Wire Wire Line
-	6450 6000 7100 6000
-Wire Wire Line
-	6800 6000 6800 5900
-Wire Wire Line
-	6800 5400 7100 5400
-Wire Wire Line
-	7800 3050 7800 2950
-Connection ~ 8250 3900
-Wire Wire Line
-	8250 2950 8250 3900
-Connection ~ 7950 3700
-Wire Wire Line
-	7950 2950 7950 3700
-Wire Wire Line
-	8800 4400 8800 4000
-Wire Wire Line
-	8800 4000 9000 4000
-Wire Wire Line
-	9000 3600 8600 3600
-Wire Wire Line
-	9000 3900 7250 3900
-Wire Wire Line
-	9000 4150 8800 4150
-Connection ~ 8800 4150
-Wire Wire Line
-	8100 2950 8100 3800
-Connection ~ 8100 3800
-Wire Wire Line
-	8600 2050 7950 2050
-Wire Wire Line
-	7950 2050 7950 2200
-Wire Wire Line
-	8600 3600 8600 2000
-Connection ~ 8600 2050
-Wire Wire Line
-	6800 5500 6800 5300
-Connection ~ 6800 5400
-Wire Wire Line
-	9000 5400 9100 5400
-Wire Wire Line
-	10000 5450 10000 5400
-Wire Wire Line
-	10000 5400 9700 5400
-Connection ~ 9800 5400
-Wire Wire Line
-	10000 6050 10000 5850
-Connection ~ 10000 6000
-Wire Wire Line
-	8100 7650 8100 7200
-Wire Wire Line
-	7800 8100 7800 8300
-Connection ~ 7800 8300
-Wire Wire Line
-	6800 6600 6800 8300
-Connection ~ 6800 8300
-Wire Wire Line
-	10300 6600 9000 6600
-Wire Wire Line
-	8300 7200 8300 7550
-Wire Wire Line
-	8300 7550 8550 7550
-Wire Wire Line
-	8550 7550 8550 7650
-Wire Wire Line
-	9850 8300 9850 7100
-Wire Wire Line
-	9250 7350 7100 7350
-Connection ~ 7900 7350
-Wire Wire Line
-	5750 3800 9000 3800
-Wire Wire Line
-	9800 5500 9800 5400
-$Comp
-L SI2333DS Q?
-U 1 1 51138AE6
-P 9500 4950
-F 0 "Q?" H 9160 5370 60  0000 R CNN
-F 1 "SI2333DS" H 9460 5275 60  0000 R CNN
-	1    9500 4950
-	1    0    0    -1
-$EndComp
+	5750 6400 7100 6400
+Text HLabel 5750 3900 0    60   Output ~ 0
+USB_ID
+Text HLabel 5750 6400 0    60   Output ~ 0
+ENABLE_USB_OTH
+$Comp
+L 0VD #PWR?
+U 1 1 5118C7E6
+P 6800 6200
+F 0 "#PWR?" H 6860 6315 50  0001 L CNN
+F 1 "0VD" H 6730 6140 50  0000 L CNN
+	1    6800 6200
+	1    0    0    -1
+$EndComp
+Text HLabel 10300 6400 2    60   Output ~ 0
+BAT_PWR_FAULT
+Text HLabel 10300 6300 2    60   Output ~ 0
+BAT_CHARGE
+Text HLabel 10300 6200 2    60   Output ~ 0
+USB_VBUS_GOOD
 Text HLabel 5750 3800 0    60   BiDi ~ 0
 USB_D+
@@
 U 1 1 51125812
 P 7100 7100
-F 0 "R?" H 7220 7150 50  0000 C CNN
-F 1 "R" H 7200 7050 50  0000 C CNN
+F 0 "R?" H 7250 7150 50  0000 C CNN
+F 1 "100k" H 7300 7050 50  0000 C CNN
 	1    7100 7100
 	1    0    0    -1
@@
 L 0VD #PWR?
 U 1 1 51125703
-P 6450 8550
-F 0 "#PWR?" H 6510 8665 50  0001 L CNN
-F 1 "0VD" H 6380 8490 50  0000 L CNN
-	1    6450 8550
+P 6800 8500
+F 0 "#PWR?" H 6860 8615 50  0001 L CNN
+F 1 "0VD" H 6730 8440 50  0000 L CNN
+	1    6800 8500
 	1    0    0    -1
 $EndComp
@@
 U 1 1 511256F7
 P 8550 7900
-F 0 "R?" H 8670 7950 50  0000 C CNN
-F 1 "R" H 8650 7850 50  0000 C CNN
+F 0 "R?" H 8700 7950 50  0000 C CNN
+F 1 "1k" H 8700 7850 50  0000 C CNN
 	1    8550 7900
 	1    0    0    -1
@@
 U 1 1 511256F0
 P 8100 7900
-F 0 "R?" H 8220 7950 50  0000 C CNN
-F 1 "R" H 8200 7850 50  0000 C CNN
+F 0 "R?" H 8250 7950 50  0000 C CNN
+F 1 "3k01" H 8300 7850 50  0000 C CNN
 	1    8100 7900
 	1    0    0    -1
@@
 L C C?
 U 1 1 511256E0
-P 7800 7900
-F 0 "C?" H 7850 8000 50  0000 L CNN
-F 1 "C" H 7850 7800 50  0000 L CNN
-	1    7800 7900
+P 7500 7900
+F 0 "C?" H 7550 8000 50  0000 L CNN
+F 1 "100n" H 7500 7800 50  0000 L CNN
+	1    7500 7900
 	1    0    0    -1
 $EndComp
@@
 L 0VD #PWR?
 U 1 1 511256BE
-P 10000 6200
-F 0 "#PWR?" H 10060 6315 50  0001 L CNN
-F 1 "0VD" H 9930 6140 50  0000 L CNN
-	1    10000 6200
+P 9450 6100
+F 0 "#PWR?" H 9510 6215 50  0001 L CNN
+F 1 "0VD" H 9380 6040 50  0000 L CNN
+	1    9450 6100
 	1    0    0    -1
 $EndComp
@@
 L +5V_USB #PWR?
 U 1 1 5112560B
-P 6800 5150
-F 0 "#PWR?" H 6825 5080 50  0001 L CNN
-F 1 "+5V_USB" H 6665 5215 50  0000 L CNN
-	1    6800 5150
+P 6800 5200
+F 0 "#PWR?" H 6825 5130 50  0001 L CNN
+F 1 "+5V_USB" H 6665 5265 50  0000 L CNN
+	1    6800 5200
 	1    0    0    -1
 $EndComp
@@
 L +5V_USB #PWR?
 U 1 1 511255D3
-P 8600 1850
-F 0 "#PWR?" H 8625 1780 50  0001 L CNN
-F 1 "+5V_USB" H 8465 1915 50  0000 L CNN
-	1    8600 1850
-	1    0    0    -1
-$EndComp
+P 8600 1900
+F 0 "#PWR?" H 8625 1830 50  0001 L CNN
+F 1 "+5V_USB" H 8465 1965 50  0000 L CNN
+	1    8600 1900
+	1    0    0    -1
+$EndComp

Commit message: wip
Parts:
- added C?: 100n, symbol C
- added U?: LTC2942-1, symbol LTC2942-1
Connections:
- net labels added: +V_BAT_OR_USB, BAT_GG_SCL, BAT_GG_SDA, BAT_GG_~AL~/CC
- wire segments 52 -> 58
Other:
- note added: "Connect PAD to insulated thermal relief plane"

Commit message: wip
Connections:
- net labels removed: 0VBAT
- wire segments 58 -> 56
Other:
- note added: "Connect PAD to isolated thermal relief plane"
- note removed: "Connect PAD to insulated thermal relief plane"
